File: PCB/Motor_Driver/Motor_Driver.brd (EAGLE design)
At the start: 41.9 x 47.9 mm, 17 parts, among them IC1 L298, X1 22-23-2021, X2 22-23-2021

Commit message: Updated the control PCBA design
Other:
- board text added: "By Tao Liu"
Changed lines of the file:
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@@
 </layers>
 <board>
+<fusionsync huburn="a.YnVzaW5lc3M6aG90bWFpbDIzMzg1Mw" projecturn="a.YnVzaW5lc3M6aG90bWFpbDIzMzg1MyNEMjAyMTAzMjMzOTYxNDQxODE" f3durn="urn:adsk.wipprod:dm.lineage:9UXUGBF-TiKeN7ydi89aGQ" pcbguid="7d8327c6-94c0-4d39-908f-29e6094fccd7" lastpulledtime="" lastsyncedchangeguid="" latestrevisionid="be8198b9-3118-40b5-be4f-77ad47b6fb1c" lastsyncedrevisionid="be8198b9-3118-40b5-be4f-77ad47b6fb1c" lastboardhashguid="77621194-82e3-f3d6-67e3-7bd5955036f6" lastpushedtime="2021-04-07T08:10:26Z" linktopcb3d="true"/>
 <plain>
 <wire x1="-1.27" y1="2.54" x2="40.62" y2="2.54" width="0" layer="20"/>
@@
 <wire x1="40.62" y1="50.47" x2="-1.27" y2="50.47" width="0" layer="20"/>
 <wire x1="-1.27" y1="50.47" x2="-1.27" y2="2.54" width="0" layer="20"/>
+<text x="2.54" y="6.35" size="1.778" layer="25" rot="R90">By Tao Liu</text>
 </plain>
 <attributes>
@@
 </note>
 <note version="8.3" severity="warning">
+Since Version 8.3, EAGLE supports Fusion synchronisation.
+This feature will not be available in this version and saving
+the document will break the link to the Fusion PCB feature.
+</note>
+<note version="8.3" severity="warning">
